Commit message: modified the urdf to include top plate and rpi

File: urdf/spider.urdf (robot description, URDF)
Before this commit: robot spiderbytes_v1, 28 links, 27 joints
Links:
- removed link battery_holder
- removed link link_bracket_rotation_1
- removed link link_bracket_rotation_2
- removed link link_bracket_rotation_3
- removed link link_bracket_rotation_4
- removed link link_motor_1_1
- removed link link_motor_1_2
- removed link link_motor_1_3
- removed link link_motor_2_1
- removed link link_motor_2_2
- removed link link_motor_2_3
- removed link link_motor_3_1
- removed link link_motor_3_2
- removed link link_motor_3_3
- removed link link_motor_4_1
- removed link link_motor_4_2
- removed link link_motor_4_3
- removed link pwm_board
- removed link rpi4b
- added link link-servo_4_1, mass 0.00241193943906811; collision mesh filename=file://$(find spiderbytes)/meshes/link-servo_4_1.STL; visual mesh filename=file://$(find spiderbytes)/meshes/link-servo_4_1.STL
- added link link_battery, mass 0.045114; collision mesh filename=file://$(find spiderbytes)/meshes/link_battery.STL; visual mesh filename=file://$(find spiderbytes)/meshes/link_battery.STL
- added link link_pwm, mass 0.00798764310040845; collision mesh filename=file://$(find spiderbytes)/meshes/link_pwm.STL; visual mesh filename=file://$(find spiderbytes)/meshes/link_pwm.STL
- added link link_rotation_1, mass 0.00723872418872687; collision mesh filename=file://$(find spiderbytes)/meshes/link_rotation_1.STL; visual mesh filename=file://$(find spiderbytes)/meshes/link_rotation_1.STL
- added link link_rotation_2, mass 0.00723872418872687; collision mesh filename=file://$(find spiderbytes)/meshes/link_rotation_2.STL; visual mesh filename=file://$(find spiderbytes)/meshes/link_rotation_2.STL
- added link link_rotation_3, mass 0.00723872418872688; collision mesh filename=file://$(find spiderbytes)/meshes/link_rotation_3.STL; visual mesh filename=file://$(find spiderbytes)/meshes/link_rotation_3.STL
- added link link_rotation_4, mass 0.00723872418872688; collision mesh filename=file://$(find spiderbytes)/meshes/link_rotation_4.STL; visual mesh filename=file://$(find spiderbytes)/meshes/link_rotation_4.STL
- added link link_rpi, mass 0.0186966914652476; collision mesh filename=file://$(find spiderbytes)/meshes/link_rpi.STL; visual mesh filename=file://$(find spiderbytes)/meshes/link_rpi.STL
- added link link_servo_1_1, mass 0.00241193943982337; collision mesh filename=file://$(find spiderbytes)/meshes/link_servo_1_1.STL; visual mesh filename=file://$(find spiderbytes)/meshes/link_servo_1_1.STL
- added link link_servo_1_2, mass 0.00241193943485351; collision mesh filename=file://$(find spiderbytes)/meshes/link_servo_1_2.STL; visual mesh filename=file://$(find spiderbytes)/meshes/link_servo_1_2.STL
- added link link_servo_1_3, mass 0.00241193942630469; collision mesh filename=file://$(find spiderbytes)/meshes/link_servo_1_3.STL; visual mesh filename=file://$(find spiderbytes)/meshes/link_servo_1_3.STL
- added link link_servo_2_1, mass 0.00241193943974115; collision mesh filename=file://$(find spiderbytes)/meshes/link_servo_2_1.STL; visual mesh filename=file://$(find spiderbytes)/meshes/link_servo_2_1.STL
- added link link_servo_2_2, mass 0.00241193943297475; collision mesh filename=file://$(find spiderbytes)/meshes/link_servo_2_2.STL; visual mesh filename=file://$(find spiderbytes)/meshes/link_servo_2_2.STL
- added link link_servo_2_3, mass 0.00241193942492555; collision mesh filename=file://$(find spiderbytes)/meshes/link_servo_2_3.STL; visual mesh filename=file://$(find spiderbytes)/meshes/link_servo_2_3.STL
- added link link_servo_3_1, mass 0.00241193943993923; collision mesh filename=file://$(find spiderbytes)/meshes/link_servo_3_1.STL; visual mesh filename=file://$(find spiderbytes)/meshes/link_servo_3_1.STL
- added link link_servo_3_2, mass 0.00241193945679526; collision mesh filename=file://$(find spiderbytes)/meshes/link_servo_3_2.STL; visual mesh filename=file://$(find spiderbytes)/meshes/link_servo_3_2.STL
- added link link_servo_3_3, mass 0.00241193944354092; collision mesh filename=file://$(find spiderbytes)/meshes/link_servo_3_3.STL; visual mesh filename=file://$(find spiderbytes)/meshes/link_servo_3_3.STL
- added link link_servo_4_2, mass 0.00241193947314956; collision mesh filename=file://$(find spiderbytes)/meshes/link_servo_4_2.STL; visual mesh filename=file://$(find spiderbytes)/meshes/link_servo_4_2.STL
- added link link_servo_4_3, mass 0.00241193947200566; collision mesh filename=file://$(find spiderbytes)/meshes/link_servo_4_3.STL; visual mesh filename=file://$(find spiderbytes)/meshes/link_servo_4_3.STL
- added link link_top_plate, mass 0.0217679973832744; collision mesh filename=file://$(find spiderbytes)/meshes/link_top_plate.STL; visual mesh filename=file://$(find spiderbytes)/meshes/link_top_plate.STL
- link base_link: mass 0.034039 -> 0.0340388036693426
Joints:
- removed joint battery_joint_fixed
- removed joint joint_bracket_1
- removed joint joint_bracket_2
- removed joint joint_bracket_3
- removed joint joint_bracket_4
- removed joint joint_motor_1_1
- removed joint joint_motor_1_2
- removed joint joint_motor_1_3
- removed joint joint_motor_2_1
- removed joint joint_motor_2_2
- removed joint joint_motor_2_3
- removed joint joint_motor_3_1
- removed joint joint_motor_3_2
- removed joint joint_motor_3_3
- removed joint joint_motor_4_1
- removed joint joint_motor_4_2
- removed joint joint_motor_4_3
- removed joint pwn_joint_fixed
- removed joint rpi_joint_fixed
- added joint joint_battery: type fixed, parent base_link, child link_battery, origin xyz=0.10368 -0.053893 0.023072 rpy=-1.5708 0 1.5708, axis 0 0 0
- added joint joint_pwm: type fixed, parent base_link, child link_pwm, origin xyz=0.039197 -0.068612 0.038017 rpy=-1.5708 0 -1.5708, axis 0 0 0
- added joint joint_rotation_1: type revolute, parent base_link, child link_rotation_1, origin xyz=0.078161 -0.10758 0.031017 rpy=-1.5708 0 2.3807, axis 0 1 0, limit lower=-1.5708 upper=1.5708 effort=10 velocity=100
- added joint joint_rotation_2: type revolute, parent base_link, child link_rotation_2, origin xyz=0.078161 -0.029647 0.031017 rpy=-1.5708 0 -2.3281, axis 0 1 0, limit lower=-1.5708 upper=1.5708 effort=10 velocity=100
- added joint joint_rotation_3: type revolute, parent base_link, child link_rotation_3, origin xyz=0.00023248 -0.029647 0.031017 rpy=-1.5708 0 -0.80128, axis 0 1 0, limit lower=-1.5708 upper=1.5708 effort=10 velocity=100
- added joint joint_rotation_4: type revolute, parent base_link, child link_rotation_4, origin xyz=0.00023248 -0.10758 0.031017 rpy=-1.5708 0 0.73985, axis 0 1 0, limit lower=-1.5708 upper=1.5708 effort=10 velocity=100
- added joint joint_rpi: type fixed, parent link_top_plate, child link_rpi, origin xyz=-0.01 0.0101 -0.0245 rpy=0 0 0, axis 0 0 0
- added joint joint_servo_1_1: type fixed, parent link_rotation_1, child link_servo_1_1, origin xyz=-0.0055 -0.025 0 rpy=3.1416 0 0, axis 0 0 0
- added joint joint_servo_1_2: type fixed, parent link_rotation_1, child link_servo_1_2, origin xyz=-0.0385 -0.0145 0.011 rpy=-1.5708 0 0, axis 0 0 0
- added joint joint_servo_1_3: type fixed, parent link_leg_1, child link_servo_1_3, origin xyz=-0.00525 0.004 -0.0005 rpy=-3.1416 0 0, axis 0 0 0
- added joint joint_servo_2_1: type fixed, parent link_rotation_2, child link_servo_2_1, origin xyz=-0.0055 -0.025 0 rpy=3.1416 0 0, axis 0 0 0
- added joint joint_servo_2_2: type fixed, parent link_rotation_2, child link_servo_2_2, origin xyz=-0.0385 -0.0145 0.004 rpy=-1.5708 0 0, axis 0 0 0
- added joint joint_servo_2_3: type fixed, parent link_leg_2, child link_servo_2_3, origin xyz=-0.00525 0.011 0.0005 rpy=3.1416 0 0, axis 0 0 0
- added joint joint_servo_3_1: type fixed, parent link_rotation_3, child link_servo_3_1, origin xyz=-0.0055 -0.025 0 rpy=3.1416 0 0, axis 0 0 0
- added joint joint_servo_3_2: type fixed, parent link_rotation_3, child link_servo_3_2, origin xyz=-0.0385 -0.0145 -0.0065 rpy=-1.5708 0 0, axis 0 0 0
- added joint joint_servo_3_3: type fixed, parent link_leg_3, child link_servo_3_3, origin xyz=-0.00525 -0.0065 -0.0005 rpy=3.1416 0 0, axis 0 0 0
- added joint joint_servo_4_1: type fixed, parent link_rotation_4, child link-servo_4_1, origin xyz=-0.0055 -0.0145 0 rpy=3.1416 0 0, axis 0 0 0
- added joint joint_servo_4_2: type fixed, parent link_rotation_4, child link_servo_4_2, origin xyz=-0.0385 -0.0145 0.011 rpy=-1.5708 0 0, axis 0 0 0
- added joint joint_servo_4_3: type fixed, parent link_leg_4, child link_servo_4_3, origin xyz=-0.00525 0.004 -0.0005 rpy=-3.1416 0 0, axis 0 0 0
- added joint joint_top_plate: type fixed, parent base_link, child link_top_plate, origin xyz=0.039197 -0.068612 0.067017 rpy=1.5708 0 0, axis 0 0 0
- joint joint_leg_2: origin xyz=-0.0077121 0.0063658 0.01 rpy=1.5708 0 2.4702 -> xyz=0.071 0 0 rpy=1.5708 0 2.4702
- joint joint_leg_4: origin xyz=0.066765 0.0035088 0 rpy=1.5708 0 2.4512 -> xyz=0.071 0 0 rpy=1.5708 0 2.4512
- joint joint_limb_1: parent link_bracket_rotation_1 -> link_rotation_1
- joint joint_limb_2: origin xyz=-0.0385 -0.0145 0.001 rpy=0 0 -2.4515 -> xyz=-0.033 -0.0145 0 rpy=0 0 -2.4515; parent link_bracket_rotation_2 -> link_rotation_2
- joint joint_limb_3: parent link_bracket_rotation_3 -> link_rotation_3
- joint joint_limb_4: origin xyz=-0.0385 -0.0145 0.001 rpy=0 0 -2.4497 -> xyz=-0.033 -0.0145 0 rpy=0 0 -2.4497; parent link_bracket_rotation_4 -> link_rotation_4
