Commit message: added variables, formations

File: urdf/spidey_v7.xacro (robot description, xacro)
@@ -48,5 +48,5 @@
     <origin xyz="0.2 0.15 0" rpy="0 0 1.5708"/>
     <axis xyz="0 0 1"/>
-    <limit lower="-1.57" upper="1.57" effort="10" velocity="2"/>
+    <limit lower="-1.57" upper="1.57" effort="100" velocity="100"/>
   </joint>
   <!-- THIGH -->
@@ -77,5 +77,5 @@
     <origin xyz="0.025 0 0"/>
     <axis xyz="0 1 0"/>
-    <limit lower="-1.5708" upper="1.5708" effort="10" velocity="2"/>
+    <limit lower="-1.5708" upper="1.5708" effort="100" velocity="100"/>
   </joint>
   <!-- LEG -->
@@ -106,5 +106,5 @@
     <origin xyz="0.2 0 0"/>
     <axis xyz="0 1 0"/>
-    <limit lower="-1.5708" upper="1.5708" effort="10" velocity="2"/>
+    <limit lower="-1.5708" upper="1.5708" effort="100" velocity="100"/>
   </joint>
   <!-- FRONT RIGHT -->
@@ -114,5 +114,5 @@
     <origin xyz="0.2 -0.15 0" rpy="0 0 -1.5708"/>
     <axis xyz="0 0 1"/>
-    <limit lower="-1.5708" upper="1.5708" effort="10" velocity="2"/>
+    <limit lower="-1.5708" upper="1.5708" effort="100" velocity="100"/>
   </joint>
   <link name="hip_fr">
@@ -142,5 +142,5 @@
     <origin xyz="0.025 0 0"/>
     <axis xyz="0 1 0"/>
-    <limit lower="-1.5708" upper="1.5708" effort="10" velocity="2"/>
+    <limit lower="-1.5708" upper="1.5708" effort="100" velocity="100"/>
   </joint>
   <link name="thigh_fr"><visual><origin xyz="0.1 0 0" rpy="0 1.5708 0"/><geometry><cylinder radius="0.025" length="0.2"/></geometry></visual>
@@ -166,5 +166,5 @@
     <origin xyz="0.2 0 0"/>
     <axis xyz="0 1 0"/>
-    <limit lower="-1.5708" upper="1.5708" effort="10" velocity="2"/>
+    <limit lower="-1.5708" upper="1.5708" effort="100" velocity="100"/>
   </joint>
   <link name="leg_fr"><visual><origin xyz="0 0 -0.15"/><geometry><cylinder radius="0.02" length="0.3"/></geometry></visual>
@@ -191,5 +191,5 @@
     <origin xyz="-0.2 0.15 0" rpy="0 0 1.5708"/>
     <axis xyz="0 0 1"/>
-    <limit lower="-1.5708" upper="1.5708" effort="10" velocity="2"/>
+    <limit lower="-1.5708" upper="1.5708" effort="100" velocity="100"/>
   </joint>
   <link name="hip_rl"><visual><geometry><cylinder radius="0.03" length="0.05"/></geometry></visual>
@@ -214,5 +214,5 @@
     <origin xyz="0.025 0 0"/>
     <axis xyz="0 1 0"/>
-    <limit lower="-1.5708" upper="1.5708" effort="10" velocity="2"/>
+    <limit lower="-1.5708" upper="1.5708" effort="100" velocity="100"/>
   </joint>
   <link name="thigh_rl"><visual><origin xyz="0.1 0 0" rpy="0 1.5708 0"/><geometry><cylinder radius="0.025" length="0.2"/></geometry></visual>
@@ -238,5 +238,5 @@
     <origin xyz="0.2 0 0"/>
     <axis xyz="0 1 0"/>
-    <limit lower="-1.5708" upper="1.5708" effort="10" velocity="2"/>
+    <limit lower="-1.5708" upper="1.5708" effort="100" velocity="100"/>
   </joint>
   <link name="leg_rl"><visual><origin xyz="0 0 -0.15"/><geometry><cylinder radius="0.02" length="0.3"/></geometry></visual>
@@ -263,5 +263,5 @@
     <origin xyz="-0.2 -0.15 0" rpy="0 0 -1.5708"/>
     <axis xyz="0 0 1"/>
-    <limit lower="-1.5708" upper="1.5708" effort="10" velocity="2"/>
+    <limit lower="-1.5708" upper="1.5708" effort="100" velocity="100"/>
   </joint>
   <link name="hip_rr"><visual><geometry><cylinder radius="0.03" length="0.05"/></geometry></visual>
@@ -286,5 +286,5 @@
     <origin xyz="0.025 0 0"/>
     <axis xyz="0 1 0"/>
-    <limit lower="-1.5708" upper="1.5708" effort="10" velocity="2"/>
+    <limit lower="-1.5708" upper="1.5708" effort="100" velocity="100"/>
   </joint>
   <link name="thigh_rr"><visual><origin xyz="0.1 0 0" rpy="0 1.5708 0"/><geometry><cylinder radius="0.025" length="0.2"/></geometry></visual>
@@ -310,5 +310,5 @@
     <origin xyz="0.2 0 0"/>
     <axis xyz="0 1 0"/>
-    <limit lower="-1.5708" upper="1.5708" effort="10" velocity="2"/>
+    <limit lower="-1.5708" upper="1.5708" effort="100" velocity="100"/>
   </joint>
   <link name="leg_rr"><visual><origin xyz="0 0 -0.15"/><geometry><cylinder radius="0.02" length="0.3"/></geometry></visual>
