Commit message: modified moment of inertia for robot

File: urdf/spidey_v8.xacro (robot description, xacro)
@@ -108,5 +108,5 @@
   </collision>
   <inertial>
-    <origin xyz="0 0 0" rpy="1.5708 0 0"/>
+    <origin xyz="0 0 0" rpy="0 1.5708 0"/>
     <mass value="0.25"/>
     <inertia
@@ -208,5 +208,5 @@
   </collision>
   <inertial>
-    <origin xyz="0 0 0"/>
+    <origin xyz="0 0 0" rpy="0 1.5708 0"/>
     <mass value="0.25"/>
     <inertia
@@ -300,5 +300,5 @@
   </collision>
   <inertial>
-    <origin xyz="0 0 0"/>
+    <origin xyz="0 0 0" rpy="0 1.5708 0"/>
     <mass value="0.25"/>
     <inertia
@@ -392,5 +392,5 @@
   </collision>
   <inertial>
-    <origin xyz="0 0 0"/>
+    <origin xyz="0 0 0" rpy="0 1.5708 0"/>
     <mass value="0.25"/>
     <inertia

Commit message: modified z position of 4 legs

File: urdf/spidey_v8.xacro (robot description, xacro)
@@ -122,5 +122,5 @@
     <parent link="thigh_fl"/>
     <child link="leg_fl"/>
-    <origin xyz="0.045 0 -0.01"/>
+    <origin xyz="0.045 0 -0.045"/>
     <axis xyz="0 1 0"/>
     <limit lower="-1.5708" upper="1.5708" effort="100" velocity="100"/>
@@ -191,5 +191,5 @@
     <parent link="thigh_fr"/>
     <child link="leg_fr"/>
-    <origin xyz="0.045 0 -0.01"/>
+    <origin xyz="0.045 0 -0.045"/>
     <axis xyz="0 1 0"/>
     <limit lower="-1.5708" upper="1.5708" effort="100" velocity="100"/>
@@ -283,5 +283,5 @@
     <parent link="thigh_rl"/>
     <child link="leg_rl"/>
-       <origin xyz="0.045 0 -0.01"/>
+       <origin xyz="0.045 0 -0.045"/>
     <axis xyz="0 1 0"/>
     <limit lower="-1.5708" upper="1.5708" effort="100" velocity="100"/>
@@ -375,5 +375,5 @@
     <parent link="thigh_rr"/>
     <child link="leg_rr"/>
-        <origin xyz="0.045 0 -0.01"/>
+        <origin xyz="0.045 0 -0.045"/>
     <axis xyz="0 1 0"/>
     <limit lower="-1.5708" upper="1.5708" effort="100" velocity="100"/>

Commit message: modified gait controller

File: urdf/spidey_v8.xacro (robot description, xacro)
@@ -403,8 +403,108 @@
   </inertial>
   </link>
-  <gazebo reference="leg_fl"><mu1>1.2</mu1><mu2>1.2</mu2></gazebo>
-  <gazebo reference="leg_fr"><mu1>1.2</mu1><mu2>1.2</mu2></gazebo>
-  <gazebo reference="leg_rr"><mu1>1.2</mu1><mu2>1.2</mu2></gazebo>
-  <gazebo reference="leg_rr"><mu1>1.2</mu1><mu2>1.2</mu2></gazebo>
+<link name="foot_fl">
+  <collision>
+    <!-- Put it at the tip/bottom of your leg -->
+    <origin xyz="0.040 0 -0.105" rpy="0 0 0"/>
+    <geometry>
+      <sphere radius="0.018"/>
+    </geometry>
+  </collision>
+  <visual>
+    <origin xyz="0.040 0 -0.105" rpy="0 0 0"/>
+    <geometry>
+      <sphere radius="0.018"/>
+    </geometry>
+  </visual>
+  <inertial>
+    <mass value="0.02"/>
+    <inertia ixx="1e-5" iyy="1e-5" izz="1e-5" ixy="0" ixz="0" iyz="0"/>
+  </inertial>
+</link>
+<joint name="foot_joint_fl" type="fixed">
+  <parent link="leg_fl"/>
+  <child link="foot_fl"/>
+  <origin xyz="0 0 0" rpy="0 0 0"/>
+</joint>
+<link name="foot_fr">
+  <collision>
+    <!-- Put it at the tip/bottom of your leg -->
+    <origin xyz="0.040 0 -0.105" rpy="0 0 0"/>
+    <geometry>
+      <sphere radius="0.018"/>
+    </geometry>
+  </collision>
+  <visual>
+    <origin xyz="0.040 0 -0.105" rpy="0 0 0"/>
+    <geometry>
+      <sphere radius="0.018"/>
+    </geometry>
+  </visual>
+  <inertial>
+    <mass value="0.02"/>
+    <inertia ixx="1e-5" iyy="1e-5" izz="1e-5" ixy="0" ixz="0" iyz="0"/>
+  </inertial>
+</link>
+<joint name="foot_joint_fr" type="fixed">
+  <parent link="leg_fr"/>
+  <child link="foot_fr"/>
+  <origin xyz="0 0 0" rpy="0 0 0"/>
+</joint>
+<link name="foot_rl">
+  <collision>
+    <!-- Put it at the tip/bottom of your leg -->
+    <origin xyz="0.040 0 -0.105" rpy="0 0 0"/>
+    <geometry>
+      <sphere radius="0.018"/>
+    </geometry>
+  </collision>
+  <visual>
+    <origin xyz="0.040 0 -0.105" rpy="0 0 0"/>
+    <geometry>
+      <sphere radius="0.018"/>
+    </geometry>
+  </visual>
+  <inertial>
+    <mass value="0.02"/>
+    <inertia ixx="1e-5" iyy="1e-5" izz="1e-5" ixy="0" ixz="0" iyz="0"/>
+  </inertial>
+</link>
+<joint name="foot_joint_rl" type="fixed">
+  <parent link="leg_rl"/>
+  <child link="foot_rl"/>
+  <origin xyz="0 0 0" rpy="0 0 0"/>
+</joint>
+<link name="foot_rr">
+  <collision>
+    <!-- Put it at the tip/bottom of your leg -->
+    <origin xyz="0.040 0 -0.105" rpy="0 0 0"/>
+    <geometry>
+      <sphere radius="0.018"/>
+    </geometry>
+  </collision>
+  <visual>
+    <origin xyz="0.040 0 -0.105" rpy="0 0 0"/>
+    <geometry>
+      <sphere radius="0.018"/>
+    </geometry>
+  </visual>
+  <inertial>
+    <mass value="0.02"/>
+    <inertia ixx="1e-5" iyy="1e-5" izz="1e-5" ixy="0" ixz="0" iyz="0"/>
+  </inertial>
+</link>
+<joint name="foot_joint_rr" type="fixed">
+  <parent link="leg_rr"/>
+  <child link="foot_rr"/>
+  <origin xyz="0 0 0" rpy="0 0 0"/>
+</joint>
+  <!-- <gazebo reference="leg_fl"><mu1>5</mu1><mu2>5</mu2></gazebo>
+  <gazebo reference="leg_fr"><mu1>5</mu1><mu2>5</mu2></gazebo>
+  <gazebo reference="leg_rr"><mu1>5</mu1><mu2>5</mu2></gazebo>
+  <gazebo reference="leg_rl"><mu1>5</mu1><mu2>5</mu2></gazebo> -->
+    <gazebo reference="foot_fl"><mu1>5</mu1><mu2>5</mu2></gazebo>
+  <gazebo reference="foot_fr"><mu1>5</mu1><mu2>5</mu2></gazebo>
+  <gazebo reference="foot_rr"><mu1>5</mu1><mu2>5</mu2></gazebo>
+  <gazebo reference="foot_rl"><mu1>5</mu1><mu2>5</mu2></gazebo>
   <ros2_control name="spiderbytes_system" type="system">
     <hardware>

Commit message: added wheels at the bottom of legs

File: urdf/spidey_v8.xacro (robot description, xacro)
@@ -406,13 +406,15 @@
   <collision>
     <!-- Put it at the tip/bottom of your leg -->
-    <origin xyz="0.040 0 -0.105" rpy="0 0 0"/>
-    <geometry>
-      <sphere radius="0.018"/>
+    <!-- <origin xyz="0.040 0 -0.105" rpy="0 0 0"/> -->
+    <geometry>
+    <!-- <sphere radius="0.018" /> -->
+      <cylinder radius="0.018" length="0.01"/>
     </geometry>
   </collision>
   <visual>
-    <origin xyz="0.040 0 -0.105" rpy="0 0 0"/>
-    <geometry>
-      <sphere radius="0.018"/>
+    <!-- <origin xyz="0.040 0 -0.105" rpy="0 0 0"/> -->
+    <geometry>
+    <!-- <sphere radius="0.018" /> -->
+     <cylinder radius="0.018" length="0.01"/>
     </geometry>
   </visual>
@@ -422,28 +424,72 @@
   </inertial>
 </link>
-<joint name="foot_joint_fl" type="fixed">
+<link name="foot_fr">
+  <collision>
+    <!-- Put it at the tip/bottom of your leg -->
+    <!-- <origin xyz="0.040 0 -0.105" rpy="0 0 0"/> -->
+    <geometry>
+    <!-- <sphere radius="0.018" /> -->
+     <cylinder radius="0.018" length="0.01"/>
+    </geometry>
+  </collision>
+  <visual>
+    <!-- <origin xyz="0.040 0 -0.105" rpy="0 0 0"/> -->
+    <geometry>
+    <!-- <sphere radius="0.018" /> -->
+      <cylinder radius="0.018" length="0.01"/>
+    </geometry>
+  </visual>
+  <inertial>
+    <mass value="0.02"/>
+    <inertia ixx="1e-5" iyy="1e-5" izz="1e-5" ixy="0" ixz="0" iyz="0"/>
+  </inertial>
+</link>
+<link name="foot_rl">
+  <collision>
+    <!-- Put it at the tip/bottom of your leg -->
+    <!-- <origin xyz="0.040 0 -0.105" rpy="0 0 0"/> -->
+    <geometry>
+    <!-- <sphere radius="0.018" /> -->
+      <cylinder radius="0.018" length="0.01"/>
+    </geometry>
+  </collision>
+  <visual>
+    <!-- <origin xyz="0.040 0 -0.105" rpy="0 0 0"/> -->
+    <geometry>
+    <!-- <sphere radius="0.018" /> -->
+     <cylinder radius="0.018" length="0.01"/>
+    </geometry>
+  </visual>
+  <inertial>
+    <mass value="0.02"/>
+    <inertia ixx="1e-5" iyy="1e-5" izz="1e-5" ixy="0" ixz="0" iyz="0"/>
+  </inertial>
+</link>
+<link name="foot_rr">
+  <collision>
+    <!-- Put it at the tip/bottom of your leg -->
+    <!-- <origin xyz="0.040 0 -0.105" rpy="0 0 0"/> -->
+    <geometry>
+    <!-- <sphere radius="0.018" /> -->
+     <cylinder radius="0.018" length="0.01"/>
+    </geometry>
+  </collision>
+  <visual>
+    <!-- <origin xyz="0.040 0 -0.105" rpy="0 0 0"/> -->
+    <geometry>
+    <!-- <sphere radius="0.018" /> -->
+      <cylinder radius="0.018" length="0.01"/>
+    </geometry>
+  </visual>
+  <inertial>
+    <mass value="0.02"/>
+    <inertia ixx="1e-5" iyy="1e-5" izz="1e-5" ixy="0" ixz="0" iyz="0"/>
+  </inertial>
+</link>
+<!-- <joint name="foot_joint_fl" type="fixed">
   <parent link="leg_fl"/>
   <child link="foot_fl"/>
   <origin xyz="0 0 0" rpy="0 0 0"/>
 </joint>
-<link name="foot_fr">
-  <collision>
-    <!-- Put it at the tip/bottom of your leg -->
-    <origin xyz="0.040 0 -0.105" rpy="0 0 0"/>
-    <geometry>
-      <sphere radius="0.018"/>
-    </geometry>
-  </collision>
-  <visual>
-    <origin xyz="0.040 0 -0.105" rpy="0 0 0"/>
-    <geometry>
-      <sphere radius="0.018"/>
-    </geometry>
-  </visual>
-  <inertial>
-    <mass value="0.02"/>
-    <inertia ixx="1e-5" iyy="1e-5" izz="1e-5" ixy="0" ixz="0" iyz="0"/>
-  </inertial>
-</link>
 <joint name="foot_joint_fr" type="fixed">
   <parent link="leg_fr"/>
@@ -451,23 +497,4 @@
   <origin xyz="0 0 0" rpy="0 0 0"/>
 </joint>
-<link name="foot_rl">
-  <collision>
-    <!-- Put it at the tip/bottom of your leg -->
-    <origin xyz="0.040 0 -0.105" rpy="0 0 0"/>
-    <geometry>
-      <sphere radius="0.018"/>
-    </geometry>
-  </collision>
-  <visual>
-    <origin xyz="0.040 0 -0.105" rpy="0 0 0"/>
-    <geometry>
-      <sphere radius="0.018"/>
-    </geometry>
-  </visual>
-  <inertial>
-    <mass value="0.02"/>
-    <inertia ixx="1e-5" iyy="1e-5" izz="1e-5" ixy="0" ixz="0" iyz="0"/>
-  </inertial>
-</link>
 <joint name="foot_joint_rl" type="fixed">
   <parent link="leg_rl"/>
@@ -475,27 +502,32 @@
   <origin xyz="0 0 0" rpy="0 0 0"/>
 </joint>
-<link name="foot_rr">
-  <collision>
-    <!-- Put it at the tip/bottom of your leg -->
-    <origin xyz="0.040 0 -0.105" rpy="0 0 0"/>
-    <geometry>
-      <sphere radius="0.018"/>
-    </geometry>
-  </collision>
-  <visual>
-    <origin xyz="0.040 0 -0.105" rpy="0 0 0"/>
-    <geometry>
-      <sphere radius="0.018"/>
-    </geometry>
-  </visual>
-  <inertial>
-    <mass value="0.02"/>
-    <inertia ixx="1e-5" iyy="1e-5" izz="1e-5" ixy="0" ixz="0" iyz="0"/>
-  </inertial>
-</link>
 <joint name="foot_joint_rr" type="fixed">
   <parent link="leg_rr"/>
   <child link="foot_rr"/>
   <origin xyz="0 0 0" rpy="0 0 0"/>
+</joint> -->
+<joint name="foot_joint_fl" type="continuous">
+  <parent link="leg_fl"/>
+  <child link="foot_fl"/>
+  <axis xyz="1 0 0"/>
+  <origin xyz="0.040 0 -0.105" rpy="0 0 0"/>
+</joint>
+<joint name="foot_joint_fr" type="continuous">
+  <parent link="leg_fr"/>
+  <child link="foot_fr"/>
+  <axis xyz="-1 0 0"/>
+  <origin xyz="0.040 0 -0.105" rpy="0 0 0"/>
+</joint>
+<joint name="foot_joint_rl" type="continuous">
+  <parent link="leg_rl"/>
+  <child link="foot_rl"/>
+  <axis xyz="1 0 0"/>
+  <origin xyz="0.040 0 -0.105" rpy="0 0 0"/>
+</joint>
+<joint name="foot_joint_rr" type="continuous">
+  <parent link="leg_rr"/>
+  <child link="foot_rr"/>
+  <axis xyz="-1 0 0"/>
+  <origin xyz="0.040 0 -0.105" rpy="0 0 0"/>
 </joint>
   <!-- <gazebo reference="leg_fl"><mu1>5</mu1><mu2>5</mu2></gazebo>
@@ -503,8 +535,67 @@
   <gazebo reference="leg_rr"><mu1>5</mu1><mu2>5</mu2></gazebo>
   <gazebo reference="leg_rl"><mu1>5</mu1><mu2>5</mu2></gazebo> -->
-    <gazebo reference="foot_fl"><mu1>5</mu1><mu2>5</mu2></gazebo>
+  <gazebo reference="foot_fl"><mu1>5</mu1><mu2>5</mu2></gazebo>
   <gazebo reference="foot_fr"><mu1>5</mu1><mu2>5</mu2></gazebo>
   <gazebo reference="foot_rr"><mu1>5</mu1><mu2>5</mu2></gazebo>
   <gazebo reference="foot_rl"><mu1>5</mu1><mu2>5</mu2></gazebo>
+    <!-- <gazebo reference="foot_fl">
+        <mu1 value="200.0" />
+        <mu2 value="200.0" />
+        <kp  value="1000000.0" />
+        <kd  value="1.0" />
+        <minDepth>0.005</minDepth>
+    </gazebo>
+    <gazebo reference="foot_fr">
+        <mu1 value="200.0" />
+        <mu2 value="200.0" />
+        <kp  value="1000000.0" />
+        <kd  value="1.0" />
+        <minDepth>0.005</minDepth>
+    </gazebo>
+    <gazebo reference="foot_rl">
+        <mu1 value="200.0" />
+        <mu2 value="200.0" />
+        <kp  value="1000000.0" />
+        <kd  value="1.0" />
+        <minDepth>0.005</minDepth>
+    </gazebo>
+    <gazebo reference="foot_rl">
+        <mu1 value="200.0" />
+        <mu2 value="200.0" />
+        <kp  value="1000000.0" />
+        <kd  value="1.0" />
+        <minDepth>0.005</minDepth>
+    </gazebo> -->
+    <gazebo>
+        <plugin name="ignition::gazebo::systems::DiffDrive" filename="ignition-gazebo-diff-drive-system">
+            <num_wheel_pairs>2</num_wheel_pairs>
+            <!-- Wheel Information -->
+            <left_joint>foot_joint_fl</left_joint>
+            <left_joint>foot_joint_rl</left_joint>
+            <right_joint>foot_joint_fr</right_joint>
+            <right_joint>foot_joint_rr</right_joint>
+            <wheel_separation>0.26</wheel_separation>
+            <wheel_radius>0.018</wheel_radius>
+            <!-- Limits -->
+            <max_linear_acceleration>5</max_linear_acceleration>
+            <min_linear_acceleration>-5</min_linear_acceleration>
+            <max_angular_acceleration>4</max_angular_acceleration>
+            <min_angular_acceleration>-4</min_angular_acceleration>
+            <max_linear_velocity>5.0</max_linear_velocity>
+            <min_linear_velocity>-5.0</min_linear_velocity>
+            <max_angular_velocity>4.0</max_angular_velocity>
+            <min_angular_velocity>-4.0</min_angular_velocity>
+            <!-- Output -->
+            <frame_id>odom</frame_id>
+            <child_frame_id>base_link</child_frame_id>
+            <!-- Topics -->
+            <topic>/cmd_vel</topic>
+            <odom_topic>/odometry/wheels</odom_topic>
+            <tf_topic>/tf_gazebo</tf_topic>
+        </plugin>
+        <plugin filename="ignition-gazebo-joint-state-publisher-system" name="ignition::gazebo::systems::JointStatePublisher">
+            <topic>/joint_states</topic>
+        </plugin>
+    </gazebo>
   <ros2_control name="spiderbytes_system" type="system">
     <hardware>
