Commit message: corrected offsets in stl files and fixed global origin

File: urdf/spidey_v4.urdf (robot description, URDF)
Before this commit: robot spiderbytes_v4, 14 links, 13 joints
Links:
- removed link base_center
- link base_link: geometry collision mesh filename=file://$(find spiderbytes)/meshes/v4_base_link.stl; visual mesh filename=file://$(find spiderbytes)/meshes/v4_base_link.stl
- link link_leg_1: geometry collision mesh filename=file://$(find spiderbytes)/meshes/v4_link_leg_1.stl; visual mesh filename=file://$(find spiderbytes)/meshes/v4_link_leg_1.stl
- link link_leg_2: geometry collision mesh filename=file://$(find spiderbytes)/meshes/v4_link_leg_2.stl; visual mesh filename=file://$(find spiderbytes)/meshes/v4_link_leg_2.stl
- link link_leg_3: geometry collision mesh filename=file://$(find spiderbytes)/meshes/v4_link_leg_3.stl; visual mesh filename=file://$(find spiderbytes)/meshes/v4_link_leg_3.stl
- link link_leg_4: geometry collision mesh filename=file://$(find spiderbytes)/meshes/v4_link_leg_4.stl; visual mesh filename=file://$(find spiderbytes)/meshes/v4_link_leg_4.stl
- link link_limb_1: geometry collision mesh filename=file://$(find spiderbytes)/meshes/v4_link_limb_1.stl; visual mesh filename=file://$(find spiderbytes)/meshes/v4_link_limb_1.stl
- link link_limb_2: geometry collision mesh filename=file://$(find spiderbytes)/meshes/v4_link_limb_2.stl; visual mesh filename=file://$(find spiderbytes)/meshes/v4_link_limb_2.stl
- link link_limb_3: geometry collision mesh filename=file://$(find spiderbytes)/meshes/v4_link_limb_3.stl; visual mesh filename=file://$(find spiderbytes)/meshes/v4_link_limb_3.stl
- link link_limb_4: geometry collision mesh filename=file://$(find spiderbytes)/meshes/v4_link_limb_4.stl; visual mesh filename=file://$(find spiderbytes)/meshes/v4_link_limb_4.stl
- link link_rotation_1: geometry collision mesh filename=file://$(find spiderbytes)/meshes/v4_link_rotation_1.stl; visual mesh filename=file://$(find spiderbytes)/meshes/v4_link_rotation_1.stl
- link link_rotation_2: geometry collision mesh filename=file://$(find spiderbytes)/meshes/v4_link_rotation_2.stl; visual mesh filename=file://$(find spiderbytes)/meshes/v4_link_rotation_2.stl
- link link_rotation_3: geometry collision mesh filename=file://$(find spiderbytes)/meshes/v4_link_rotation_3.stl; visual mesh filename=file://$(find spiderbytes)/meshes/v4_link_rotation_3.stl
- link link_rotation_4: geometry collision mesh filename=file://$(find spiderbytes)/meshes/v4_link_rotation_4.stl; visual mesh filename=file://$(find spiderbytes)/meshes/v4_link_rotation_4.stl
Joints:
- removed joint base_center_to_base_link
- joint joint_leg_1: origin xyz=0.071 0 0 rpy=1.5708 0 2.4731 -> xyz=0.04 -0.001 0.0 rpy=1.5708 0 2.4731
- joint joint_leg_2: origin xyz=0.071 0 0 rpy=1.5708 0 2.4702 -> xyz=0.04 0.001 0.0 rpy=1.5708 0 2.4702
- joint joint_leg_3: origin xyz=0.071 0 0 rpy=1.5708 0 2.4783 -> xyz=0.04 -0.001 0.0 rpy=1.5708 0 2.4783
- joint joint_leg_4: origin xyz=0.071 0 0 rpy=1.5708 0 2.4512 -> xyz=0.04 -0.001 0.0 rpy=1.5708 0 2.4512
- joint joint_limb_1: origin xyz=-0.033 -0.0145 0 rpy=0 0 -2.4811 -> xyz=-0.04 -0.017 -0.005 rpy=0 0 -2.4811
- joint joint_limb_2: origin xyz=-0.033 -0.0145 0 rpy=0 0 -2.4515 -> xyz=-0.04 -0.017 -0.005 rpy=0 0 -2.4515
- joint joint_limb_3: origin xyz=-0.033 -0.0145 0 rpy=0 0 -2.4471 -> xyz=-0.04 -0.017 -0.005 rpy=0 0 -2.4471
- joint joint_limb_4: origin xyz=-0.033 -0.0145 0 rpy=0 0 -2.4497 -> xyz=-0.04 -0.017 -0.005 rpy=0 0 -2.4497
- joint joint_rotation_1: origin xyz=0.078161 -0.10758 0.031017 rpy=-1.5708 0 2.3807 -> xyz=0.0518161 -0.050758 -0.021017 rpy=-1.5708 0 2.3807
- joint joint_rotation_2: origin xyz=0.078161 -0.029647 0.031017 rpy=-1.5708 0 -2.3281 -> xyz=0.0518161 0.050758 -0.021017 rpy=-1.5708 0 -2.3281
- joint joint_rotation_3: origin xyz=0.00023248 -0.029647 0.031017 rpy=-1.5708 0 -0.80128 -> xyz=-0.0518161 0.050758 -0.021017 rpy=-1.5708 0 -0.80128
- joint joint_rotation_4: origin xyz=0.00023248 -0.10758 0.031017 rpy=-1.5708 0 0.73985 -> xyz=-0.0518161 -0.050758 -0.021017 rpy=-1.5708 0 0.73985
