Commit message: added joint group position controller

File: urdf/accessories/camera.urdf (robot description, URDF)
Before this commit: robot spider_camera, 2 links, 2 joints
Links:
- link camera_link: geometry collision box size=0.03 0.03 0.02; visual box size=0.06 0.03 0.01
Joints:
- joint camera_joint: origin xyz=${wheel_x_offset + 0.05} 0 0.08 rpy=0 0 0 -> xyz=${wheel_x_offset} 0 0.05 rpy=0 0 0
